File: BoardFiles/MdSDE.sch (KiCad schematic (older format))
At the start: 2 parts

Commit message: Created ComponentBrick.pro
Created Component Brick Project.  Added component library for MdSDE,
included relative search path, included library.
Added schematic component for DIP Switches “SPST_x3”
Parts:
- gave numbers to parts that had none: 2
Changed lines of the file:
@@
 $EndSheet
 $Comp
-L DIL16 P?
+L DIL16 P101
 U 1 1 56A733B1
 P 8650 1550
-F 0 "P?" H 8650 2000 50  0000 C CNN
+F 0 "P101" H 8650 2000 50  0000 C CNN
 F 1 "DIL16" V 8650 1550 50  0000 C CNN
 F 2 "" H 8650 1550 50  0000 C CNN
@@
 $EndComp
 $Comp
-L DIL16 P?
+L DIL16 P102
 U 1 1 56A73671
 P 8650 3050
-F 0 "P?" H 8650 3500 50  0000 C CNN
+F 0 "P102" H 8650 3500 50  0000 C CNN
 F 1 "DIL16" V 8650 3050 50  0000 C CNN
 F 2 "" H 8650 3050 50  0000 C CNN
@@
 	3400 5400 3650 5400
 $Comp
-L GND #PWR?
+L GND #PWR102
 U 1 1 56AE1915
 P 3000 4100
-F 0 "#PWR?" H 3000 3850 50  0001 C CNN
+F 0 "#PWR102" H 3000 3850 50  0001 C CNN
 F 1 "GND" H 3000 3950 50  0000 C CNN
 F 2 "" H 3000 4100 50  0000 C CNN
@@
 $EndComp
 $Comp
-L GND #PWR?
+L GND #PWR105
 U 1 1 56AE1B43
 P 6600 4150
-F 0 "#PWR?" H 6600 3900 50  0001 C CNN
+F 0 "#PWR105" H 6600 3900 50  0001 C CNN
 F 1 "GND" H 6600 4000 50  0000 C CNN
 F 2 "" H 6600 4150 50  0000 C CNN
@@
 $EndComp
 $Comp
-L GND #PWR?
+L GND #PWR103
 U 1 1 56AE1D6A
 P 3650 7200
-F 0 "#PWR?" H 3650 6950 50  0001 C CNN
+F 0 "#PWR103" H 3650 6950 50  0001 C CNN
 F 1 "GND" H 3650 7050 50  0000 C CNN
 F 2 "" H 3650 7200 50  0000 C CNN
@@
 $EndComp
 $Comp
-L GND #PWR?
+L GND #PWR101
 U 1 1 56AE1F91
 P 3000 2250
-F 0 "#PWR?" H 3000 2000 50  0001 C CNN
+F 0 "#PWR101" H 3000 2000 50  0001 C CNN
 F 1 "GND" H 3000 2100 50  0000 C CNN
 F 2 "" H 3000 2250 50  0000 C CNN
@@
 $EndComp
 $Comp
-L GND #PWR?
+L GND #PWR104
 U 1 1 56AE21B8
 P 6600 2300
-F 0 "#PWR?" H 6600 2050 50  0001 C CNN
+F 0 "#PWR104" H 6600 2050 50  0001 C CNN
 F 1 "GND" H 6600 2150 50  0000 C CNN
 F 2 "" H 6600 2300 50  0000 C CNN
