File: BoardFiles/componentBrickSub.sch (KiCad schematic (older format))
At the start: 10 parts

Commit message: Created ComponentBrick.pro
Created Component Brick Project.  Added component library for MdSDE,
included relative search path, included library.
Added schematic component for DIP Switches “SPST_x3”
Parts:
- removed SW? (x6): SPST, symbol SPST
- added SW?: Coded_Switch, symbol Coded_Switch
- added SW? (x3): SPST_x3, symbol SPST_x3
- gave numbers to parts that had none: 4
Connections:
- wire segments 18 -> 22
