File: BoardFiles/routingBrickFilter.sch (KiCad schematic (older format))
At the start: 8 parts

Commit message: Created ComponentBrick.pro
Created Component Brick Project.  Added component library for MdSDE,
included relative search path, included library.
Added schematic component for DIP Switches “SPST_x3”
Parts:
- gave numbers to parts that had none: 8
Changed lines of the file:
@@
 $EndDescr
 $Comp
-L SPST SW?
+L SPST SW1201
 U 1 1 56A68FB8
 P 5000 2700
-F 0 "SW?" H 5000 2800 50  0000 C CNN
+F 0 "SW1201" H 5000 2800 50  0000 C CNN
 F 1 "SPST" H 5000 2600 50  0000 C CNN
 F 2 "" H 5000 2700 60  0000 C CNN
@@
 $EndComp
 $Comp
-L SPST SW?
+L SPST SW1202
 U 1 1 56A68FBF
 P 5400 2700
-F 0 "SW?" H 5400 2800 50  0000 C CNN
+F 0 "SW1202" H 5400 2800 50  0000 C CNN
 F 1 "SPST" H 5400 2600 50  0000 C CNN
 F 2 "" H 5400 2700 60  0000 C CNN
@@
 $EndComp
 $Comp
-L SPST SW?
+L SPST SW1203
 U 1 1 56A68FC6
 P 5800 2700
-F 0 "SW?" H 5800 2800 50  0000 C CNN
+F 0 "SW1203" H 5800 2800 50  0000 C CNN
 F 1 "SPST" H 5800 2600 50  0000 C CNN
 F 2 "" H 5800 2700 60  0000 C CNN
@@
 $EndComp
 $Comp
-L SPST SW?
+L SPST SW1204
 U 1 1 56A68FCD
 P 6200 2700
-F 0 "SW?" H 6200 2800 50  0000 C CNN
+F 0 "SW1204" H 6200 2800 50  0000 C CNN
 F 1 "SPST" H 6200 2600 50  0000 C CNN
 F 2 "" H 6200 2700 60  0000 C CNN
@@
 $EndComp
 $Comp
-L C C?
+L C C1201
 U 1 1 56A68FD4
 P 5000 3500
-F 0 "C?" H 5025 3600 50  0000 L CNN
+F 0 "C1201" H 5025 3600 50  0000 L CNN
 F 1 "0.1u" H 5025 3400 50  0000 L CNN
 F 2 "" H 5038 3350 30  0000 C CNN
@@
 $EndComp
 $Comp
-L C C?
+L C C1202
 U 1 1 56A68FDB
 P 5400 3500
-F 0 "C?" H 5425 3600 50  0000 L CNN
+F 0 "C1202" H 5425 3600 50  0000 L CNN
 F 1 "0.1u" H 5425 3400 50  0000 L CNN
 F 2 "" H 5438 3350 30  0000 C CNN
@@
 $EndComp
 $Comp
-L C C?
+L C C1203
 U 1 1 56A68FE2
 P 5800 3500
-F 0 "C?" H 5825 3600 50  0000 L CNN
+F 0 "C1203" H 5825 3600 50  0000 L CNN
 F 1 "0.1u" H 5825 3400 50  0000 L CNN
 F 2 "" H 5838 3350 30  0000 C CNN
@@
 $EndComp
 $Comp
-L C C?
+L C C1204
 U 1 1 56A68FE9
 P 6200 3500
-F 0 "C?" H 6225 3600 50  0000 L CNN
+F 0 "C1204" H 6225 3600 50  0000 L CNN
 F 1 "0.1u" H 6225 3400 50  0000 L CNN
 F 2 "" H 6238 3350 30  0000 C CNN
@@
 Connection ~ 5800 3650
 $Comp
-L GND #PWR?
+L GND #PWR1201
 U 1 1 56A68FF7
 P 5600 3750
-F 0 "#PWR?" H 5600 3500 50  0001 C CNN
+F 0 "#PWR1201" H 5600 3500 50  0001 C CNN
 F 1 "GND" H 5600 3600 50  0000 C CNN
 F 2 "" H 5600 3750 60  0000 C CNN
