File: BoardFiles/MdSDE_ComponentBrick/ComponentBrickSub.sch (KiCad schematic (older format))
At the start: 6 parts, among them SW201 Coded_Switch, SW202 SPST_x3

Commit message: Updated footprints
Reduced size of bounding rectangle on components
Parts:
- RV201: footprint (none) -> Footprints:3314_Potentiometer
- SW201: footprint (none) -> Footprints:SH-7000RotarySwitch
Changed lines of the file:
@@
 AR Path="/56D62CF7/56D61280" Ref="RV801"  Part="1"
 AR Path="/56D62CFC/56D61280" Ref="RV901"  Part="1"
-F 0 "RV901" H 7200 2750 50  0000 C CNN
+F 0 "RV201" H 7200 2750 50  0000 C CNN
 F 1 "POT" H 7200 2850 50  0000 C CNN
-F 2 "" H 7200 2850 60  0001 C CNN
+F 2 "Footprints:3314_Potentiometer" H 7200 2850 60  0001 C CNN
 F 3 "" H 7200 2850 60  0000 C CNN
 	1    7200 2850
@@
 AR Path="/56D62CF7/56D612B4" Ref="SW801"  Part="1"
 AR Path="/56D62CFC/56D612B4" Ref="SW901"  Part="1"
-F 0 "SW901" H 3250 3650 50  0000 C CNN
+F 0 "SW201" H 3250 3650 50  0000 C CNN
 F 1 "Coded_Switch" H 3150 2951 50  0000 C CNN
-F 2 "" H 3150 3300 60  0001 C CNN
+F 2 "Footprints:SH-7000RotarySwitch" H 3150 3300 60  0001 C CNN
 F 3 "" H 3150 3300 60  0000 C CNN
 	1    3150 3300
@@
 AR Path="/56D62CF7/56D6142F" Ref="C803"  Part="1"
 AR Path="/56D62CFC/56D6142F" Ref="C903"  Part="1"
-F 0 "C903" H 4610 3970 50  0000 L CNN
+F 0 "C203" H 4610 3970 50  0000 L CNN
 F 1 "C_Small" H 4610 3820 50  0000 L CNN
 F 2 "Capacitors_SMD:C_1206_HandSoldering" H 4600 3900 60  0001 C CNN
@@
 AR Path="/56D62CF7/56D6147F" Ref="C802"  Part="1"
 AR Path="/56D62CFC/56D6147F" Ref="C902"  Part="1"
-F 0 "C902" H 4310 3970 50  0000 L CNN
+F 0 "C202" H 4310 3970 50  0000 L CNN
 F 1 "C_Small" H 4310 3820 50  0000 L CNN
 F 2 "Capacitors_SMD:C_1206_HandSoldering" H 4300 3900 60  0001 C CNN
@@
 AR Path="/56D62CF7/56D614A7" Ref="C801"  Part="1"
 AR Path="/56D62CFC/56D614A7" Ref="C901"  Part="1"
-F 0 "C901" H 4010 3970 50  0000 L CNN
+F 0 "C201" H 4010 3970 50  0000 L CNN
 F 1 "C_Small" H 4010 3820 50  0000 L CNN
 F 2 "Capacitors_SMD:C_1206_HandSoldering" H 4000 3900 60  0001 C CNN
@@
 Connection ~ 4250 2550
 $Comp
-L GND #PWR201
+L GND #PWR013
 U 1 1 56D615B3
 P 5200 5000
-AR Path="/56D61275/56D615B3" Ref="#PWR201"  Part="1"
-AR Path="/56D61AB8/56D615B3" Ref="#PWR301"  Part="1"
-AR Path="/56D620FB/56D615B3" Ref="#PWR401"  Part="1"
-AR Path="/56D62100/56D615B3" Ref="#PWR501"  Part="1"
-AR Path="/56D62CED/56D615B3" Ref="#PWR601"  Part="1"
-AR Path="/56D62CF2/56D615B3" Ref="#PWR701"  Part="1"
-AR Path="/56D62CF7/56D615B3" Ref="#PWR801"  Part="1"
-AR Path="/56D62CFC/56D615B3" Ref="#PWR901"  Part="1"
-F 0 "#PWR901" H 5200 4750 50  0001 C CNN
+AR Path="/56D61275/56D615B3" Ref="#PWR013"  Part="1"
+AR Path="/56D61AB8/56D615B3" Ref="#PWR014"  Part="1"
+AR Path="/56D620FB/56D615B3" Ref="#PWR015"  Part="1"
+AR Path="/56D62100/56D615B3" Ref="#PWR016"  Part="1"
+AR Path="/56D62CED/56D615B3" Ref="#PWR017"  Part="1"
+AR Path="/56D62CF2/56D615B3" Ref="#PWR018"  Part="1"
+AR Path="/56D62CF7/56D615B3" Ref="#PWR019"  Part="1"
+AR Path="/56D62CFC/56D615B3" Ref="#PWR020"  Part="1"
+F 0 "#PWR013" H 5200 4750 50  0001 C CNN
 F 1 "GND" H 5200 4850 50  0000 C CNN
 F 2 "" H 5200 5000 60  0000 C CNN
@@
 AR Path="/56D62CF7/56D6B52C" Ref="SW802"  Part="3"
 AR Path="/56D62CFC/56D6B52C" Ref="SW902"  Part="3"
-F 0 "SW902" H 7300 2200 50  0000 C CNN
+F 0 "SW202" H 7300 2200 50  0000 C CNN
 F 1 "SPST_x3" H 7300 2000 50  0000 C CNN
 F 2 "Buttons_Switches_ThroughHole:SW_DIP_x3_Slide" H 7300 2100 60  0001 C CNN
@@
 AR Path="/56D62CF7/56D6B569" Ref="SW802"  Part="1"
 AR Path="/56D62CFC/56D6B569" Ref="SW902"  Part="1"
-F 0 "SW902" H 5450 2650 50  0000 C CNN
+F 0 "SW202" H 5450 2650 50  0000 C CNN
 F 1 "SPST_x3" H 5450 2450 50  0000 C CNN
 F 2 "Buttons_Switches_ThroughHole:SW_DIP_x3_Slide" H 5450 2550 60  0001 C CNN
@@
 AR Path="/56D62CF7/56D6B596" Ref="SW802"  Part="2"
 AR Path="/56D62CFC/56D6B596" Ref="SW902"  Part="2"
-F 0 "SW902" H 6150 3900 50  0000 C CNN
+F 0 "SW202" H 6150 3900 50  0000 C CNN
 F 1 "SPST_x3" H 6150 3700 50  0000 C CNN
 F 2 "Buttons_Switches_ThroughHole:SW_DIP_x3_Slide" H 6150 3800 60  0001 C CNN
